File: Detector inductivo-2026.kicad_pcb (KiCad board)
At the start: 2 copper layers, 95.5 x 50.5 mm, 17 parts, among them Q1 2N2222A, Q2 BC557, Q3 BC557, Q4 2N2222A

Commit message: update board
Parts:
- added H1: MountingHole, MountingHole:MountingHole_4.3x6.2mm_M4_Pad_Via, F.Cu at (80.5, 94.6)
- added H2: MountingHole, MountingHole:MountingHole_4.3x6.2mm_M4_Pad_Via, F.Cu at (80.5, 104.7)
- added H3: MountingHole, MountingHole:MountingHole_4.3x6.2mm_M4_Pad_Via, F.Cu at (80.5, 114.9)
- added H4: MountingHole, MountingHole:MountingHole_4.3x6.2mm_M4_Pad_Via, F.Cu at (80.5, 125.0)
- AE2: footprint Connector_Coaxial:BNC_TEConnectivity_1478204_Vertical -> Connector_Coaxial:SMA_Amphenol_132134-11_Vertical
- BZ1: footprint Buzzer_Beeper:MagneticBuzzer_StarMicronics_HMB -> Buzzer_Beeper:Indicator_PUI_AI-1440-TWT-24V-2-R
- moved TP2 66.2 mm to (111.0, 105.0)
- moved TP1 33.8 mm to (147.7, 105.2)
- moved R3 31.1 mm to (170.1, 96.8), turned to 180 degrees
- moved LED1 27.5 mm to (175.5, 95.2)
- moved R2 24.6 mm to (138.1, 96.8), turned to 180 degrees
- moved R4 20.3 mm to (146.7, 100.5)
- moved TP3 19.9 mm to (151.2, 96.2)
- moved R1 19.1 mm to (130.4, 100.2)
- moved Q4 17.5 mm to (158.5, 101.1)
- moved BT1 17.1 mm to (107.0, 98.0)
- moved Q2 17.1 mm to (142.2, 101.3)
- moved BZ1 15.0 mm to (187.8, 94.8)
- moved Q3 13.8 mm to (176.4, 104.0), turned to 90 degrees
- moved AE2 12.0 mm to (114.0, 99.0)
- moved R5 11.1 mm to (162.4, 100.0)
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Other:
- board size 95.5 x 50.5 mm -> 90.5 x 16.2 mm
