File: Detector inductivo-2026.kicad_sch (KiCad schematic)
At the start: 17 parts, among them Q1 2N2222A, Q2 BC557, Q3 BC557, Q4 2N2222A

Commit message: update board
Parts:
- added H1, H2, H3, H4: MountingHole, MountingHole:MountingHole_4.3x6.2mm_M4_Pad_Via, symbol Mechanical:MountingHole
- AE2: footprint Connector_Coaxial:BNC_TEConnectivity_1478204_Vertical -> Connector_Coaxial:SMA_Amphenol_132134-11_Vertical
- BZ1: footprint Buzzer_Beeper:MagneticBuzzer_StarMicronics_HMB -> Buzzer_Beeper:Indicator_PUI_AI-1440-TWT-24V-2-R
