File: _restore_backup_2026-05-18T15-43-26-205/Detector inductivo-2026.kicad_pcb (KiCad board)
At the start: 2 copper layers, 90.5 x 16.2 mm, 21 parts, among them Q1 2N2222A, Q2 BC557, Q3 BC557, Q4 2N2222A

Commit message: cambios en el pcb
Parts:
- moved BZ1 7.85 mm to (187.8, 94.8), turned to -90 degrees
- moved TP2 1.02 mm to (111.0, 105.0)
- moved TP1 0.75 mm to (147.7, 105.2)
Routing:
- net Net-(Q2-B): track 13.9 -> 0.00 mm
- net Net-(Q4-B): track 12.0 -> 0.00 mm
- net /9V: track 82.2 -> 70.7 mm
- net Net-(BZ1-+): track 10.8 -> 0.00 mm
- net Net-(Q1-C): track 9.87 -> 0.00 mm
- net Net-(AE2-A): track 8.76 -> 0.00 mm
- net Net-(Q4-C): track 7.53 -> 0.00 mm
- net Net-(Q3-B): track 6.98 -> 0.00 mm
- net Net-(LED1-K): track 6.06 -> 0.00 mm
- net Net-(Q2-C): track 4.78 -> 0.00 mm
- removed copper zone on B.Cu, net GND
