File: _restore_backup_2026-05-18T16-57-39-245/Detector inductivo-2026.kicad_pcb (KiCad board)
At the start: 2 copper layers, 90.5 x 16.2 mm, 21 parts, among them Q1 2N2222A, Q2 BC557, Q3 BC557, Q4 2N2222A

Commit message: cambios en el pcb
Parts:
- moved BZ1 7.85 mm to (187.8, 94.8), turned to -90 degrees
- moved TP1 0.75 mm to (147.7, 105.2)
Routing:
- net Net-(Q4-B): track 12.0 -> 0.00 mm
- net /9V: track 82.2 -> 70.7 mm
- net Net-(BZ1-+): track 10.8 -> 0.00 mm
- net Net-(Q4-C): track 7.53 -> 0.00 mm
- net Net-(Q3-B): track 6.98 -> 0.00 mm
- net Net-(LED1-K): track 6.06 -> 0.00 mm
- net Net-(Q2-B): track 13.9 -> 9.01 mm
- net Net-(Q2-C): track 4.78 -> 0.00 mm
- removed copper zone on B.Cu, net GND
Changed lines of the file:
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@@
 	(footprint "TestPoint:TestPoint_Bridge_Pitch2.54mm_Drill0.7mm"
 		(layer "F.Cu")
-		(at 147.73 104.5)
+		(at 147.73 105.25)
 		(descr "wire loop as test point, pitch 2.0mm, hole diameter 0.7mm, wire diameter 0.5mm")
 		(tags "test point wire loop")
@@
 		(tags "Resistor Axial_DIN0207 series Axial Horizontal pin pitch 7.62mm 0.25W = 1/4W length 6.3mm diameter 2.5mm")
 		(property "Reference" "R4"
-			(at 2.31 -2.5 0)
+			(at 3.81 2.25 0)
 			(layer "F.SilkS")
 			(effects
@@
 		)
 		(fp_text user "${REFERENCE}"
-			(at 2.31 -2.5 0)
+			(at 3.81 2.25 0)
 			(layer "F.Fab")
 			(effects
@@
 	(footprint "Buzzer_Beeper:Indicator_PUI_AI-1440-TWT-24V-2-R"
 		(layer "F.Cu")
-		(at 186.5 102.5 90)
+		(at 187.75 94.75 -90)
 		(descr "14mm Indicator, https://www.puiaudio.com/media/SpecSheet/AI-1440-TWT-24V-2-R.pdf")
 		(tags "piezo buzzer self drive oscillator")
@@
 		)
 		(property "Value" "Buzzer"
-			(at -3.5 -5 0)
+			(at 10.5 6 0)
 			(layer "F.Fab")
 			(effects
@@
 		)
 		(property "Datasheet" ""
-			(at 0 0 90)
+			(at 0 0 270)
 			(unlocked yes)
 			(layer "F.Fab")
@@
 		)
 		(property "Description" "Buzzer, polarized"
-			(at 0 0 90)
+			(at 0 0 270)
 			(unlocked yes)
 			(layer "F.Fab")
@@
 		)
 		(pad "1" thru_hole roundrect
-			(at 0 0 90)
+			(at 0 0 270)
 			(size 1.7 1.7)
 			(drill 0.9)
@@
 		)
 		(pad "2" thru_hole circle
-			(at 7.6 0 90)
+			(at 7.6 0 270)
 			(size 1.7 1.7)
 			(drill 0.9)
@@
 	)
 	(segment
-		(start 126.75 96.25)
-		(end 122.79 96.25)
-		(width 0.6)
-		(layer "B.Cu")
-		(net "Net-(Q1-C)")
-	)
-	(segment
-		(start 126.75 96.25)
-		(end 126.75 96.62)
+		(start 126.71 96.21)
+		(end 126.75 96.25)
 		(width 0.6)
 		(layer "B.Cu")
@@
 	)
 	(segment
-		(start 122.79 96.25)
-		(end 122.75 96.21)
+		(start 122.75 96.21)
+		(end 126.71 96.21)
 		(width 0.6)
 		(layer "B.Cu")
@@
 	(segment
 		(start 126.75 96.25)
-		(end 127 96.5)
+		(end 126.75 96.62)
 		(width 0.6)
 		(layer "B.Cu")
@@
 	)
 	(segment
-		(start 151.23 96.25)
-		(end 153.77 96.25)
-		(width 0.6)
-		(layer "B.Cu")
-		(net "Net-(Q4-B)")
-	)
-	(segment
-		(start 156.27 98.54)
-		(end 154.31 100.5)
-		(width 0.6)
-		(layer "B.Cu")
-		(net "Net-(Q4-B)")
-	)
-	(segment
-		(start 153.77 99.96)
-		(end 154.31 100.5)
-		(width 0.6)
-		(layer "B.Cu")
-		(net "Net-(Q4-B)")
-	)
-	(segment
-		(start 153.77 96.25)
-		(end 153.77 99.96)
-		(width 0.6)
-		(layer "B.Cu")
-		(net "Net-(Q4-B)")
-	)
-	(segment
-		(start 158.5 98.54)
-		(end 156.27 98.54)
-		(width 0.6)
-		(layer "B.Cu")
-		(net "Net-(Q4-B)")
-	)
-	(segment
-		(start 114 104.46)
+		(start 112 105)
 		(end 114.54 105)
 		(width 0.6)
@@
 	(segment
 		(start 114.54 105)
-		(end 112 105)
+		(end 114.04 105)
 		(width 0.6)
 		(layer "B.Cu")
@@
 	)
 	(segment
-		(start 114 99)
-		(end 114 104.46)
+		(start 114.04 105)
+		(end 114 104.96)
 		(width 0.6)
 		(layer "B.Cu")
@@
 	)
 	(segment
-		(start 142.25 101.33)
-		(end 145.86 101.33)
-		(width 0.6)
-		(layer "B.Cu")
-		(net "Net-(Q2-C)")
-	)
-	(segment
-		(start 145.86 101.33)
-		(end 146.69 100.5)
-		(width 0.6)
-		(layer "B.Cu")
-		(net "Net-(Q2-C)")
-	)
-	(segment
-		(start 142.25 98.79)
-		(end 139.46 98.79)
+		(start 114 104.96)
+		(end 114 99)
 		(width 0.6)
 		(layer "B.Cu")
-		(net "Net-(Q2-B)")
-	)
-	(segment
-		(start 130.44 96.75)
-		(end 134.5 96.75)
-		(width 0.6)
-		(layer "B.Cu")
-		(net "Net-(Q2-B)")
+		(net "Net-(AE2-A)")
 	)
 	(segment
@@
 	)
 	(segment
-		(start 139.46 98.79)
-		(end 138 100.25)
+		(start 130.44 96.75)
+		(end 134.5 96.75)
 		(width 0.6)
 		(layer "B.Cu")
@@
 	)
 	(segment
-		(start 175.5 92.71)
-		(end 177 94.21)
-		(width 0.8)
-		(layer "B.Cu")
-		(net "/9V")
-	)
-	(segment
 		(start 107 97.98)
 		(end 112.27 92.71)
@@
 	)
 	(segment
-		(start 177 94.21)
-		(end 177 98.32)
-		(width 0.8)
-		(layer "B.Cu")
-		(net "/9V")
-	)
-	(segment
 		(start 112.27 92.71)
 		(end 175.5 92.71)
@@
 		(net "/9V")
 	)
-	(segment
-		(start 177 98.32)
-		(end 176.36 98.96)
-		(width 0.8)
-		(layer "B.Cu")
-		(net "/9V")
-	)
-	(segment
-		(start 142.25 96.25)
-		(end 138.56 96.25)
-		(width 0.8)
-		(layer "B.Cu")
-		(net "/9V")
-	)
-	(segment
-		(start 138.56 96.25)
-		(end 138.06 96.75)
-		(width 0.8)
-		(layer "B.Cu")
-		(net "/9V")
-	)
-	(segment
-		(start 162.38 96.81)
-		(end 162.44 96.75)
-		(width 0.6)
-		(layer "B.Cu")
-		(net "Net-(Q4-C)")
-	)
-	(segment
-		(start 159.25 96.75)
-		(end 158.5 96)
-		(width 0.6)
-		(layer "B.Cu")
-		(net "Net-(Q4-C)")
-	)
-	(segment
-		(start 162.44 96.75)
-		(end 159.25 96.75)
-		(width 0.6)
-		(layer "B.Cu")
-		(net "Net-(Q4-C)")
-	)
-	(segment
-		(start 162.38 100)
-		(end 162.38 96.81)
-		(width 0.6)
-		(layer "B.Cu")
-		(net "Net-(Q4-C)")
-	)
-	(segment
-		(start 176.36 104.04)
-		(end 184.96 104.04)
-		(width 0.6)
-		(layer "B.Cu")
-		(net "Net-(BZ1-+)")
-	)
-	(segment
-		(start 184.96 104.04)
-		(end 186.5 102.5)
-		(width 0.6)
-		(layer "B.Cu")
-		(net "Net-(BZ1-+)")
-	)
-	(segment
-		(start 170.06 96.75)
-		(end 174 96.75)
-		(width 0.6)
-		(layer "B.Cu")
-		(net "Net-(LED1-K)")
-	)
-	(segment
-		(start 174 96.75)
-		(end 175.5 95.25)
-		(width 0.6)
-		(layer "B.Cu")
-		(net "Net-(LED1-K)")
-	)
-	(segment
-		(start 170 100)
-		(end 174.86 100)
-		(width 0.6)
-		(layer "B.Cu")
-		(net "Net-(Q3-B)")
-	)
-	(segment
-		(start 174.86 100)
-		(end 176.36 101.5)
-		(width 0.6)
-		(layer "B.Cu")
-		(net "Net-(Q3-B)")
-	)
-	(zone
-		(net "GND")
-		(layer "B.Cu")
-		(hatch edge 0.5)
-		(connect_pads
-			(clearance 0.5)
-		)
-		(min_thickness 0.25)
-		(fill yes
-			(thermal_gap 0.5)
-			(thermal_bridge_width 0.5)
-			(island_removal_mode 0)
-		)
-		(polygon
-			(pts
-				(xy 105 90.5) (xy 195.5 90.5) (xy 195.5 106.5) (xy 105 106.5)
-			)
-		)
-	)
 	(embedded_fonts no)
